File: hw/_saved_esb.sch (KiCad schematic (older format))
At the start: 2 parts, among them J101 AMPSEAL_8_POS_1-776276-1, J102 AMPSEAL_23_POS_1-776228-1

Commit message: 3.0.0 ready to order
Changed lines of the file:
@@
 F12 "SENSE3" O R 6350 7350 60
 F13 "SENSE4" O R 6350 7450 60
-F14 "VDD" I L 5450 6650 60
 $EndSheet
 Text Label 3550 6950 0    60   ~ 0
