File: hw/_saved_lpc1549.sch (KiCad schematic (older format))
At the start: 15 parts, among them J301 ARM_JTAG_SWD_HEADER_10_PINSMD, U301 MCP2551_SOIC8, X301 XTAL_7A-12.000MAAJ-T

Commit message: 3.0.0 ready to order
Parts:
- gave numbers to parts that had none: 1
Connections:
- net AC: now also U302.P$62 (PIO0_27/ACMP_I1); no longer U302.P$63 (PIO0_28/ACMP1_I3)
- net AC_SENSE: now also U302.P$4 (PIO1_0/ADC0_8); no longer U302.P$6 (PIO0_2/ADC0_6/SCT1_OUT3)
- net ALT_IG: now also U302.P$9 (PIO0_5/ADC0_3); no longer U302.P$17 (PIO0_18/SCT0_OUT5)
- net GLOW_PLUGS: now also U302.P$64 (PIO0_29/ACMP2_I3/SCT2_OUT4); no longer U302.P$62 (PIO0_27/ACMP_I1)
- net GLOW_PLUGS_SENSE: now also U302.P$2 (PIO0_0/ADC0_10/SCT0_OUT3); no longer U302.P$3 (PIO0_31/ADC0_9)
- net MOTOR_ON: now also U302.P$61 (PIO0_26/ACMP0_I3/SCT3_OUT3); no longer U302.P$16 (PIO0_9/ADC1_1/TDI)
- net MOTOR_ON_SENSE: now also U302.P$5 (PIO0_1/ADC0_7/SCT0_OUT4); no longer U302.P$7 (PIO0_3/ADC0_5/SCT1_OUT4)
- net MOTOR_START: now also U302.P$6 (PIO0_2/ADC0_6/SCT1_OUT3); no longer U302.P$15 (PIO1_1/ADC1_0)
- net MOTOR_START_SENSE: now also U302.P$7 (PIO0_3/ADC0_5/SCT1_OUT4); no longer U302.P$8 (PIO0_4/ADC0_4)
- net PUMP: now also U302.P$8 (PIO0_4/ADC0_4); no longer U302.P$19 (PIO0_10/ADC1_2)
- net PUMP_SENSE: now also U302.P$11 (PIO0_7/ADC0_1); no longer U302.P$9 (PIO0_5/ADC0_3)
- net STARTER: now also U302.P$63 (PIO0_28/ACMP1_I3); no longer U302.P$61 (PIO0_26/ACMP0_I3/SCT3_OUT3)
- net STARTER_SENSE: now also U302.P$3 (PIO0_31/ADC0_9); no longer U302.P$4 (PIO1_0/ADC0_8)
- net VDD_SENSE: now also U302.P$1 (PIO0_30/ADC0_11); no longer U302.P$2 (PIO0_0/ADC0_10/SCT0_OUT3)
Changed lines of the file:
@@
 $EndComp
 $Comp
-L +3V3 #PWR303
+L +3V3 #PWR013
 U 1 1 57E689A3
 P 3600 3950
-F 0 "#PWR303" H 3600 3800 50  0001 C CNN
+F 0 "#PWR013" H 3600 3800 50  0001 C CNN
 F 1 "+3V3" H 3615 4123 50  0000 C CNN
 F 2 "" H 3600 3950 50  0000 C CNN
@@
 $EndComp
 $Comp
-L GND #PWR304
+L GND #PWR014
 U 1 1 57E689C9
 P 3600 4550
-F 0 "#PWR304" H 3600 4300 50  0001 C CNN
+F 0 "#PWR014" H 3600 4300 50  0001 C CNN
 F 1 "GND" H 3605 4377 50  0000 C CNN
 F 2 "" H 3600 4550 50  0000 C CNN
@@
 $EndComp
 $Comp
-L GND #PWR306
+L GND #PWR015
 U 1 1 57E697A1
 P 8000 3100
-F 0 "#PWR306" H 8000 2850 50  0001 C CNN
+F 0 "#PWR015" H 8000 2850 50  0001 C CNN
 F 1 "GND" H 8005 2927 50  0000 C CNN
 F 2 "" H 8000 3100 50  0000 C CNN
@@
 $EndComp
 $Comp
-L GND #PWR305
+L GND #PWR016
 U 1 1 57E69A8B
 P 7300 3350
-F 0 "#PWR305" H 7300 3100 50  0001 C CNN
+F 0 "#PWR016" H 7300 3100 50  0001 C CNN
 F 1 "GND" H 7305 3177 50  0000 C CNN
 F 2 "" H 7300 3350 50  0000 C CNN
@@
 $EndComp
 $Comp
-L GND #PWR307
+L GND #PWR017
 U 1 1 5891FBFB
 P 9700 4500
-F 0 "#PWR307" H 9700 4250 50  0001 C CNN
+F 0 "#PWR017" H 9700 4250 50  0001 C CNN
 F 1 "GND" H 9705 4327 50  0000 C CNN
 F 2 "" H 9700 4500 50  0000 C CNN
@@
 $EndComp
 $Comp
-L +3V3 #PWR308
+L +3V3 #PWR018
 U 1 1 5891FCDE
 P 9750 3450
-F 0 "#PWR308" H 9750 3300 50  0001 C CNN
+F 0 "#PWR018" H 9750 3300 50  0001 C CNN
 F 1 "+3V3" H 9765 3623 50  0000 C CNN
 F 2 "" H 9750 3450 50  0000 C CNN
@@
 Text HLabel 7500 2050 2    60   Input ~ 0
 ALT_P/RPM
-Text HLabel 4800 2350 0    60   Input ~ 0
+Text HLabel 4800 2250 0    60   Input ~ 0
 GLOW_PLUGS_SENSE
-Text HLabel 7300 5550 2    60   Output ~ 0
+Text HLabel 7300 5750 2    60   Output ~ 0
 GLOW_PLUGS
 Wire Wire Line
@@
 	7000 2350 7500 2350
 Wire Wire Line
-	7000 5550 7300 5550
+	7000 5750 7300 5750
 Wire Wire Line
 	7000 1950 7500 1950
@@
 $EndComp
 $Comp
-L +5V #PWR301
+L +5V #PWR019
 U 1 1 58C01582
 P 2800 2750
-F 0 "#PWR301" H 2800 2600 50  0001 C CNN
+F 0 "#PWR019" H 2800 2600 50  0001 C CNN
 F 1 "+5V" H 2815 2923 50  0000 C CNN
 F 2 "" H 2800 2750 50  0000 C CNN
@@
 $EndComp
 $Comp
-L GND #PWR302
+L GND #PWR020
 U 1 1 58C01588
 P 2800 3300
-F 0 "#PWR302" H 2800 3050 50  0001 C CNN
+F 0 "#PWR020" H 2800 3050 50  0001 C CNN
 F 1 "GND" H 2805 3127 50  0000 C CNN
 F 2 "" H 2800 3300 50  0000 C CNN
@@
 CAN_RX
 Wire Wire Line
-	7000 5450 7300 5450
-Text HLabel 7300 5450 2    60   Output ~ 0
+	7000 5650 7300 5650
+Text HLabel 7300 5650 2    60   Output ~ 0
 STARTER
 Wire Wire Line
 	5200 5750 4700 5750
-Text HLabel 4800 2450 0    60   Input ~ 0
+Text HLabel 4800 2350 0    60   Input ~ 0
 STARTER_SENSE
 Wire Wire Line
 	5200 5550 4700 5550
 Wire Wire Line
-	5200 5250 4700 5250
-Text HLabel 4700 5250 0    60   Output ~ 0
+	5200 2950 4800 2950
+Text HLabel 4800 2950 0    60   Output ~ 0
 ALT_IG
 Text HLabel 4700 5550 0    60   Input ~ 0
@@
 HYDR_OIL_TEMP
 Wire Wire Line
-	5200 2350 4800 2350
+	5200 2250 4800 2250
 Text HLabel 7500 2350 2    60   Input ~ 0
 FUEL_LEVEL
 Wire Wire Line
-	5200 2450 4800 2450
+	5200 2350 4800 2350
 Text HLabel 4700 5750 0    60   Input ~ 0
 MOTOR_OIL_PRESS
 Wire Wire Line
-	5200 5150 4700 5150
-Text HLabel 4700 5050 0    60   Output ~ 0
+	7000 5450 7300 5450
+Text HLabel 4800 2650 0    60   Output ~ 0
 MOTOR_START
 Wire Wire Line
-	5200 5050 4700 5050
-Text HLabel 4700 5150 0    60   Output ~ 0
+	5200 2650 4800 2650
+Text HLabel 7300 5450 2    60   Output ~ 0
 MOTOR_ON
+Text HLabel 4800 2550 0    60   Input ~ 0
+MOTOR_ON_SENSE
 Text HLabel 4800 2750 0    60   Input ~ 0
-MOTOR_ON_SENSE
-Text HLabel 4800 2850 0    60   Input ~ 0
 MOTOR_START_SENSE
 Wire Wire Line
@@
 MOTOR_WATER_TEMP
 Wire Wire Line
-	5200 5350 4700 5350
+	5200 2850 4800 2850
 Text HLabel 4800 3050 0    60   Input ~ 0
 ALT_IG_SENSE
 Wire Wire Line
-	5200 2750 4800 2750
-Wire Wire Line
-	4800 2850 5200 2850
+	5200 2550 4800 2550
+Wire Wire Line
+	4800 2750 5200 2750
 Wire Wire Line
 	5200 3050 4800 3050
 Wire Wire Line
-	4800 2950 5200 2950
-Text HLabel 4700 5350 0    60   Output ~ 0
+	4800 3150 5200 3150
+Text HLabel 4800 2850 0    60   Output ~ 0
 PUMP
-Text HLabel 4800 2950 0    60   Input ~ 0
+Text HLabel 4800 3150 0    60   Input ~ 0
 PUMP_SENSE
 $Comp
@@
 OIL_LEVEL
 Wire Wire Line
-	5200 2650 4800 2650
-Text HLabel 4800 2650 0    60   Input ~ 0
+	5200 2450 4800 2450
+Text HLabel 4800 2450 0    60   Input ~ 0
 AC_SENSE
 Wire Wire Line
-	7000 5650 7300 5650
-Text HLabel 7300 5650 2    60   Output ~ 0
+	7000 5550 7300 5550
+Text HLabel 7300 5550 2    60   Output ~ 0
 AC
 $Comp
@@
 $EndComp
 Wire Wire Line
-	5200 2250 4800 2250
-Text HLabel 4800 2250 0    60   Input ~ 0
+	5200 2150 4800 2150
+Text HLabel 4800 2150 0    60   Input ~ 0
 VDD_SENSE
 $Comp
-L LPC1549JBD64 U?
+L LPC1549JBD64 U302
 U 1 1 59C4D0FB
 P 5700 2750
-F 0 "U?" H 6100 3826 45  0000 C CNN
+F 0 "U302" H 6100 3826 45  0000 C CNN
 F 1 "LPC1549JBD64" H 5700 2750 45  0001 L BNN
 F 2 "usevolt:QFP64" H 5730 2900 20  0001 C CNN
