File: hw/currentSense3.sch (KiCad schematic (older format))
At the start: 2 parts, among them U1201 ZXCT1086

Commit message: 3.0.0 ready to order
Parts:
- removed R1301: LRMAM1206-R015FT5, usevolt:1206, symbol LRMAM1206-R015FT5
- removed U1201: ZXCT1086, usevolt:SOT-25, symbol ZXCT1086
- added R801: LRMAT2512-R004FT4, usevolt:2512, symbol LRMAT2512-R004FT4
- added U701: ZXCT1086, usevolt:SOT-25, symbol ZXCT1086
Changed lines of the file:
@@
 $Descr A4 11693 8268
 encoding utf-8
-Sheet 12 17
+Sheet 7 17
 Title "MSB current sense sheet"
 Date "2017-02-05"
@@
 $EndDescr
 $Comp
-L ZXCT1086 U1201
-U 1 1 59B98AFC
+L ZXCT1086 U701
+U 1 1 589841A1
 P 5450 3600
-AR Path="/58C7B0A8/58BE8E88/59B98AFC" Ref="U1201"  Part="1"
-AR Path="/58C7B0A8/58BE8E96/59B98AFC" Ref="U1301"  Part="1"
-F 0 "U1301" H 5425 3887 60  0000 C CNN
+AR Path="/58BE52C9/5955DE03/589841A1" Ref="U701"  Part="1"
+AR Path="/58BE52C9/59B27EDC/589841A1" Ref="U801"  Part="1"
+AR Path="/58C7B0A8/594D8B80/589841A1" Ref="U1001"  Part="1"
+AR Path="/58C7B0A8/594D8B83/589841A1" Ref="U1101"  Part="1"
+F 0 "U1101" H 5425 3887 60  0000 C CNN
 F 1 "ZXCT1086" H 5425 3781 60  0000 C CNN
 F 2 "usevolt:SOT-25" H 5100 4050 60  0001 C CNN
@@
 $EndComp
 $Comp
-L GND #PWR1202
-U 1 1 589841A8
+L GND #PWR702
+U 1 1 59B98AFD
 P 5050 4000
-AR Path="/58C7B0A8/58BE8E88/589841A8" Ref="#PWR1202"  Part="1"
-AR Path="/58C7B0A8/58BE8E96/589841A8" Ref="#PWR1302"  Part="1"
-F 0 "#PWR1302" H 5050 3750 50  0001 C CNN
+AR Path="/58BE52C9/5955DE03/59B98AFD" Ref="#PWR702"  Part="1"
+AR Path="/58BE52C9/59B27EDC/59B98AFD" Ref="#PWR802"  Part="1"
+AR Path="/58C7B0A8/594D8B80/59B98AFD" Ref="#PWR1002"  Part="1"
+AR Path="/58C7B0A8/594D8B83/59B98AFD" Ref="#PWR1102"  Part="1"
+F 0 "#PWR1102" H 5050 3750 50  0001 C CNN
 F 1 "GND" H 5055 3827 50  0000 C CNN
 F 2 "" H 5050 4000 50  0000 C CNN
@@
 $EndComp
 $Comp
-L +3V3 #PWR1201
-U 1 1 594D8B7F
+L +3V3 #PWR701
+U 1 1 59B98AFE
 P 5050 3350
-AR Path="/58C7B0A8/58BE8E88/594D8B7F" Ref="#PWR1201"  Part="1"
-AR Path="/58C7B0A8/58BE8E96/594D8B7F" Ref="#PWR1301"  Part="1"
-F 0 "#PWR1301" H 5050 3200 50  0001 C CNN
+AR Path="/58BE52C9/5955DE03/59B98AFE" Ref="#PWR701"  Part="1"
+AR Path="/58BE52C9/59B27EDC/59B98AFE" Ref="#PWR801"  Part="1"
+AR Path="/58C7B0A8/594D8B80/59B98AFE" Ref="#PWR1001"  Part="1"
+AR Path="/58C7B0A8/594D8B83/59B98AFE" Ref="#PWR1101"  Part="1"
+F 0 "#PWR1101" H 5050 3200 50  0001 C CNN
 F 1 "+3V3" H 5065 3523 50  0000 C CNN
 F 2 "" H 5050 3350 50  0000 C CNN
@@
 Connection ~ 6200 3300
 $Comp
-L LRMAM1206-R015FT5 R1301
-U 1 1 59B972DD
+L LRMAT2512-R004FT4 R801
+U 1 1 59B97E24
 P 6200 3450
-AR Path="/58C7B0A8/58BE8E96/59B972DD" Ref="R1301"  Part="1"
-AR Path="/58BE52C9/59B27EDC/59B972DD" Ref="R?"  Part="1"
-AR Path="/58C7B0A8/58BE8E88/59B972DD" Ref="R1201"  Part="1"
-F 0 "R1301" V 6208 3508 45  0000 L CNN
-F 1 "LRMAM1206-R015FT5" V 6292 3508 45  0000 L CNN
-F 2 "usevolt:1206" H 6230 3600 20  0001 C CNN
-F 3 "http://www.farnell.com/datasheets/2158958.pdf?_ga=2.185174241.912271158.1498242272-1561825231.1484148445" H 6169 3489 60  0001 C CNN
-F 4 "756-LRMAM1206R015FT5" H 6769 4089 60  0001 C CNN "2nd Source Part Number"
-F 5 "Mouser" H 6669 3989 60  0001 C CNN "2nd Source"
-F 6 "2079441" H 6569 3889 60  0001 C CNN "1st Source Part Number"
-F 7 "Farnell" H 6469 3789 60  0001 C CNN "1st Source"
-F 8 "LRMAM1206-R015FT5" H 6369 3689 60  0001 C CNN "Manufacturer Part Number"
-F 9 "WELWYN" H 6269 3589 60  0001 C CNN "Manufacturer"
+AR Path="/58BE52C9/59B27EDC/59B97E24" Ref="R801"  Part="1"
+AR Path="/58BE52C9/5955DE03/59B97E24" Ref="R701"  Part="1"
+AR Path="/58C7B0A8/594D8B80/59B97E24" Ref="R1001"  Part="1"
+AR Path="/58C7B0A8/594D8B83/59B97E24" Ref="R1101"  Part="1"
+F 0 "R1101" V 6208 3508 45  0000 L CNN
+F 1 "LRMAT2512-R004FT4" V 6292 3508 45  0000 L CNN
+F 2 "usevolt:2512" H 6230 3600 20  0001 C CNN
+F 3 "http://www.farnell.com/datasheets/2158958.pdf?_ga=2.43265772.874534928.1505194133-1862443086.1504075057" H 6169 3489 60  0001 C CNN
+F 4 "2079418" H 6569 3889 60  0001 C CNN "1st Source Part Number"
+F 5 "Farnell" H 6469 3789 60  0001 C CNN "1st Source"
+F 6 "LRMAT2512-R002FT4" H 6369 3689 60  0001 C CNN "Manufacturer Part Number"
+F 7 "WELWYN" H 6269 3589 60  0001 C CNN "Manufacturer"
 	1    6200 3450
 	0    1    1    0
