File: hw/pwr_supply_sheet.sch (KiCad schematic (older format))
At the start: 15 parts

Commit message: 3.0.0 ready to order
Parts:
- added D205: SCHOTTKY_DIODE_V40PW10C, usevolt:SlimDPAK, symbol SCHOTTKY_DIODE_V40PW10C
Connections:
- net VDD: now also D205.3 (CATHODE)
- net VIN: now also D205.1 (A1), D205.2 (A2)
Changed lines of the file:
@@
 EESchema Schematic File Version 2
+LIBS:esb-rescue
 LIBS:kemet
-LIBS:multicomp
 LIBS:usevolt
 LIBS:wurth_elektronik_LED
 LIBS:power
 LIBS:elt21300_kicad
+LIBS:yageo
 LIBS:esb-cache
 EELAYER 26 0
@@
 $Descr A4 11693 8268
 encoding utf-8
-Sheet 2 17
+Sheet 2 13
 Title "Power supply"
 Date "2016-08-20"
@@
 	6850 3600 6850 3850
 $Comp
-L +5V #PWR06
+L +5V #PWR05
 U 1 1 57B831F8
 P 6850 3600
-F 0 "#PWR06" H 6850 3450 50  0001 C CNN
+F 0 "#PWR05" H 6850 3450 50  0001 C CNN
 F 1 "+5V" H 6865 3773 50  0000 C CNN
 F 2 "" H 6850 3600 50  0000 C CNN
@@
 Connection ~ 6850 3750
 $Comp
-L +3V3 #PWR07
+L +3V3 #PWR06
 U 1 1 57B83259
 P 8600 3600
-F 0 "#PWR07" H 8600 3450 50  0001 C CNN
+F 0 "#PWR06" H 8600 3450 50  0001 C CNN
 F 1 "+3V3" H 8615 3773 50  0000 C CNN
 F 2 "" H 8600 3600 50  0000 C CNN
@@
 Wire Wire Line
 	8750 3600 8600 3600
-Text HLabel 2550 3200 2    60   Output ~ 0
+Text HLabel 2900 3200 2    60   Output ~ 0
 VDD
 Text HLabel 2700 4300 0    60   Input ~ 0
@@
 NoConn ~ 4550 4050
 $Comp
-L VDD #PWR08
+L VDD #PWR07
 U 1 1 57B9C56A
 P 3800 2100
-F 0 "#PWR08" H 3800 1950 50  0001 C CNN
+F 0 "#PWR07" H 3800 1950 50  0001 C CNN
 F 1 "VDD" H 3817 2273 50  0000 C CNN
 F 2 "" H 3800 2100 50  0000 C CNN
@@
 $EndComp
 $Comp
-L PWR_FLAG #FLG09
+L PWR_FLAG #FLG08
 U 1 1 57B9C59C
 P 3800 2300
-F 0 "#FLG09" H 3800 2395 50  0001 C CNN
+F 0 "#FLG08" H 3800 2395 50  0001 C CNN
 F 1 "PWR_FLAG" H 3800 2523 50  0000 C CNN
 F 2 "" H 3800 2300 50  0000 C CNN
@@
 	3800 2300 3800 2100
 $Comp
-L GND #PWR010
+L GND #PWR09
 U 1 1 57B9D351
 P 4300 2350
-F 0 "#PWR010" H 4300 2100 50  0001 C CNN
+F 0 "#PWR09" H 4300 2100 50  0001 C CNN
 F 1 "GND" H 4305 2177 50  0000 C CNN
 F 2 "" H 4300 2350 50  0000 C CNN
@@
 $EndComp
 $Comp
-L PWR_FLAG #FLG011
+L PWR_FLAG #FLG010
 U 1 1 57B9D3A1
 P 4300 2150
-F 0 "#FLG011" H 4300 2245 50  0001 C CNN
+F 0 "#FLG010" H 4300 2245 50  0001 C CNN
 F 1 "PWR_FLAG" H 4300 2374 50  0000 C CNN
 F 2 "" H 4300 2150 50  0000 C CNN
@@
 	4300 2150 4300 2350
 $Comp
-L GND #PWR012
+L GND #PWR011
 U 1 1 57CF1F5E
 P 2800 4500
-F 0 "#PWR012" H 2800 4250 50  0001 C CNN
+F 0 "#PWR011" H 2800 4250 50  0001 C CNN
 F 1 "GND" H 2805 4327 50  0000 C CNN
 F 2 "" H 2800 4500 50  0000 C CNN
@@
 $EndComp
 $Comp
-L GND #PWR013
+L GND #PWR012
 U 1 1 59B128CC
 P 1600 4750
-F 0 "#PWR013" H 1600 4500 50  0001 C CNN
+F 0 "#PWR012" H 1600 4500 50  0001 C CNN
 F 1 "GND" H 1605 4577 50  0000 C CNN
 F 2 "" H 1600 4750 50  0000 C CNN
@@
 $EndComp
 Wire Wire Line
-	2550 3200 2450 3200
-Wire Wire Line
-	1500 3850 1500 3150
+	2900 3200 2450 3200
+Wire Wire Line
+	1500 2650 1500 3850
 Wire Wire Line
 	1500 3150 1650 3150
@@
 	1650 3250 1500 3250
 Connection ~ 1500 3250
+$Comp
+L SCHOTTKY_DIODE_V40PW10C D205
+U 1 1 59D9089A
+P 2050 2750
+F 0 "D205" H 2050 3097 60  0000 C CNN
+F 1 "SCHOTTKY_DIODE_V40PW10C" H 2050 2991 60  0000 C CNN
+F 2 "usevolt:SlimDPAK" H 1850 2400 60  0001 C CNN
+F 3 "http://www.farnell.com/datasheets/2245239.pdf?_ga=2.16591231.874534928.1505194133-1862443086.1504075057" H 1850 2400 60  0001 C CNN
+F 4 "2535169" H 2400 3350 60  0001 C CNN "1st Source Part Number"
+F 5 "Digikey" H 2500 3450 60  0001 C CNN "2nd Source"
+F 6 "Farnell" H 2300 3250 60  0001 C CNN "1st Source"
+F 7 "V40PW10CHM3/I" H 2200 3150 60  0001 C CNN "Manufacturer Part Number"
+F 8 "V40PW10CHM3/IGICT-ND" H 2600 3550 60  0001 C CNN "2nd Source Part Number"
+F 9 "VISHAY" H 2100 3050 60  0001 C CNN "Manufacturer"
+	1    2050 2750
+	1    0    0    -1
+$EndComp
+Wire Wire Line
+	1500 2750 1650 2750
+Connection ~ 1500 3150
+Wire Wire Line
+	1500 2650 1650 2650
+Connection ~ 1500 2750
+Wire Wire Line
+	2450 2700 2750 2700
+Wire Wire Line
+	2750 2700 2750 3200
+Connection ~ 2750 3200
 $EndSCHEMATC
