File: hw/pwr_supply_sheet.sch (KiCad schematic (older format))
At the start: 16 parts

Commit message: implemnting pump propo output
Parts:
- removed C202: T491D226K035AT, kemet:7343, symbol T491D226K035AT
- removed C203: 10nF, kemet:0603, symbol 10nF
- added C202: CAP_EEE-FK1H470P, usevolt:CAP_EEE-FK1H470P, symbol CAP_EEE-FK1H470P
- added C203: 100nF, kemet:0603, symbol 100nF
- added D206: DIODE_TVS_TPSMD28A, usevolt:DO-214AB, symbol DIODE_TVS_TPSMD28A
Connections:
- wire segments 39 -> 40

Commit message: 4.2.0 created, with working propo solenoid pump driver
Parts:
- removed C202: CAP_EEE-FK1H470P, usevolt:CAP_EEE-FK1H470P, symbol CAP_EEE-FK1H470P
- removed C203: 100nF, kemet:0603, symbol 100nF
- removed D206: DIODE_TVS_TPSMD28A, usevolt:DO-214AB, symbol DIODE_TVS_TPSMD28A
- added C202: T491D226K035AT, kemet:7343, symbol T491D226K035AT
- added C203: 10nF, kemet:0603, symbol 10nF
Connections:
- wire segments 40 -> 39

Commit message: hw bugs fixed from 4.2.0 revsion
Parts:
- removed C202: T491D226K035AT, kemet:7343, symbol T491D226K035AT
- added C202: CAP_EEE-FK1H470P, usevolt:CAP_EEE-FK1H470P, symbol CAP_EEE-FK1H470P
- added D206: DIODE_TVS_TPSMD28A, usevolt:DO-214AB, symbol DIODE_TVS_TPSMD28A
Connections:
- wire segments 39 -> 41
Changed lines of the file:
@@
 $Descr A4 11693 8268
 encoding utf-8
-Sheet 2 11
+Sheet 2 13
 Title "Power supply"
 Date "2016-08-20"
@@
 P 2800 4050
 F 0 "D203" V 2892 3982 45  0000 R CNN
-F 1 "DIODE_TVS_SMBJ33A-TRDO-214AA" V 2750 4750 45  0000 R CNN
+F 1 "DIODE_TVS_SMBJ33A-TRDO-214AA" V 2750 5250 45  0000 R CNN
 F 2 "usevolt:DO-214AA" H 2830 4200 20  0001 C CNN
 F 3 "http://www.littelfuse.com/~/media/electronics/datasheets/tvs_diodes/littelfuse_tvs_diode_smbj_datasheet.pdf.pdf" H 2910 4060 60  0001 C CNN
@@
 $EndComp
 Wire Wire Line
-	8000 4300 8000 4250
-Wire Wire Line
-	6850 4300 6850 4150
-Connection ~ 8000 4300
-Wire Wire Line
-	6200 4300 6200 4150
-Connection ~ 6850 4300
-Wire Wire Line
-	5550 4300 5550 4050
-Connection ~ 6200 4300
-Wire Wire Line
-	3800 4300 3800 4150
-Connection ~ 5550 4300
-Wire Wire Line
-	3400 4300 3400 4150
-Connection ~ 3800 4300
-Wire Wire Line
-	2800 4150 2800 4500
-Connection ~ 3400 4300
+	8000 4950 8000 4250
+Wire Wire Line
+	6850 4950 6850 4150
+Connection ~ 8000 4950
+Wire Wire Line
+	6200 4950 6200 4150
+Connection ~ 6850 4950
+Wire Wire Line
+	5550 4950 5550 4050
+Connection ~ 6200 4950
+Wire Wire Line
+	3800 4950 3800 4150
+Connection ~ 5550 4950
+Wire Wire Line
+	3400 4950 3400 4150
+Connection ~ 3800 4950
+Wire Wire Line
+	2800 4150 2800 5150
+Connection ~ 3400 4950
 Connection ~ 2800 3850
 Connection ~ 3400 3850
 Wire Wire Line
-	8600 4300 8600 4150
+	8600 4950 8600 4150
 Wire Wire Line
 	8600 3600 8600 3850
@@
 	6850 3600 6850 3850
 $Comp
-L +5V #PWR205
+L +5V #PWR206
 U 1 1 57B831F8
 P 6850 3600
-F 0 "#PWR205" H 6850 3450 50  0001 C CNN
+F 0 "#PWR206" H 6850 3450 50  0001 C CNN
 F 1 "+5V" H 6865 3773 50  0000 C CNN
 F 2 "" H 6850 3600 50  0000 C CNN
@@
 Connection ~ 6850 3750
 $Comp
-L +3V3 #PWR206
+L +3V3 #PWR207
 U 1 1 57B83259
 P 8600 3600
-F 0 "#PWR206" H 8600 3450 50  0001 C CNN
+F 0 "#PWR207" H 8600 3450 50  0001 C CNN
 F 1 "+3V3" H 8615 3773 50  0000 C CNN
 F 2 "" H 8600 3600 50  0000 C CNN
@@
 Wire Wire Line
 	8750 3600 8600 3600
-Text HLabel 2900 3200 2    60   Output ~ 0
+Text HLabel 3150 2700 2    60   Output ~ 0
 VDD
-Text HLabel 2700 4300 0    60   Input ~ 0
+Text HLabel 2700 4950 0    60   Input ~ 0
 GND
-Connection ~ 2800 4300
+Connection ~ 2800 4950
 NoConn ~ 4550 3850
 NoConn ~ 4550 3950
 NoConn ~ 4550 4050
 $Comp
-L VDD #PWR203
+L VDD #PWR204
 U 1 1 57B9C56A
 P 3800 2100
-F 0 "#PWR203" H 3800 1950 50  0001 C CNN
+F 0 "#PWR204" H 3800 1950 50  0001 C CNN
 F 1 "VDD" H 3817 2273 50  0000 C CNN
 F 2 "" H 3800 2100 50  0000 C CNN
@@
 	3800 2300 3800 2100
 $Comp
-L GND #PWR204
+L GND #PWR205
 U 1 1 57B9D351
 P 4300 2350
-F 0 "#PWR204" H 4300 2100 50  0001 C CNN
+F 0 "#PWR205" H 4300 2100 50  0001 C CNN
 F 1 "GND" H 4305 2177 50  0000 C CNN
 F 2 "" H 4300 2350 50  0000 C CNN
@@
 	4300 2150 4300 2350
 $Comp
-L GND #PWR202
+L GND #PWR201
 U 1 1 57CF1F5E
-P 2800 4500
-F 0 "#PWR202" H 2800 4250 50  0001 C CNN
-F 1 "GND" H 2805 4327 50  0000 C CNN
-F 2 "" H 2800 4500 50  0000 C CNN
-F 3 "" H 2800 4500 50  0000 C CNN
-	1    2800 4500
+P 2800 5150
+F 0 "#PWR201" H 2800 4900 50  0001 C CNN
+F 1 "GND" H 2805 4977 50  0000 C CNN
+F 2 "" H 2800 5150 50  0000 C CNN
+F 3 "" H 2800 5150 50  0000 C CNN
+	1    2800 5150
 	1    0    0    -1
 $EndComp
@@
 	2000 3850 2300 3850
 Wire Wire Line
-	2700 4300 8600 4300
+	2700 4950 8600 4950
 $Comp
 L DIODE_RS07J-GS18 D201
@@
 	1    1900 3850
 	1    0    0    -1
-$EndComp
-$Comp
-L T491D226K035AT C202
-U 1 1 597AF50C
-P 3800 4050
-F 0 "C202" V 3708 4153 45  0000 L CNN
-F 1 "T491D226K035AT" V 3792 4153 45  0000 L CNN
-F 2 "kemet:7343" H 3830 4200 20  0001 C CNN
-F 3 "http://www.farnell.com/datasheets/2121523.pdf?_ga=1.259966538.1948984246.1460023966" H 3800 3990 60  0001 C CNN
-F 4 "399-8375-1-ND" H 4400 4590 60  0001 C CNN "2nd Source Part Number"
-F 5 "Farnell" H 4100 4290 60  0001 C CNN "1st Source"
-F 6 "T491D226K035AT" H 4000 4190 60  0001 C CNN "Manufacturer Part Number"
-F 7 "Digikey" H 4300 4490 60  0001 C CNN "2nd Source"
-F 8 "Kemet" H 3900 4090 60  0001 C CNN "Manufacturer"
-F 9 "1457504" H 4200 4390 60  0001 C CNN "1st Source Part Number"
-	1    3800 4050
-	0    1    1    0
 $EndComp
 $Comp
@@
 L 10K R201
 U 1 1 59B1277F
-P 1600 4050
-F 0 "R201" V 1608 4108 45  0000 L CNN
-F 1 "10K" V 1692 4108 45  0000 L CNN
-F 2 "multicomp:0603" H 1630 4200 20  0001 C CNN
-F 3 "http://www.farnell.com/datasheets/1788326.pdf?_ga=1.214208087.1948984246.1460023966" H 1569 4089 60  0001 C CNN
-F 4 "9330399" H 1969 4489 60  0001 C CNN "1st Source Part Number"
-F 5 "Farnell" H 1869 4389 60  0001 C CNN "1st Source"
-F 6 "MC0063W0603110K" H 1769 4289 60  0001 C CNN "Manufacturer Part Number"
-F 7 "MULTICOMP" H 1669 4189 60  0001 C CNN "Manufacturer"
-	1    1600 4050
+P 3100 4050
+F 0 "R201" V 3108 4108 45  0000 L CNN
+F 1 "10K" V 3192 4108 45  0000 L CNN
+F 2 "multicomp:0603" H 3130 4200 20  0001 C CNN
+F 3 "http://www.farnell.com/datasheets/1788326.pdf?_ga=1.214208087.1948984246.1460023966" H 3069 4089 60  0001 C CNN
+F 4 "9330399" H 3469 4489 60  0001 C CNN "1st Source Part Number"
+F 5 "Farnell" H 3369 4389 60  0001 C CNN "1st Source"
+F 6 "MC0063W0603110K" H 3269 4289 60  0001 C CNN "Manufacturer Part Number"
+F 7 "MULTICOMP" H 3169 4189 60  0001 C CNN "Manufacturer"
+	1    3100 4050
 	0    1    1    0
 $EndComp
@@
 L 1K R202
 U 1 1 59B12803
-P 1600 4450
-F 0 "R202" V 1608 4508 45  0000 L CNN
-F 1 "1K" V 1692 4508 45  0000 L CNN
-F 2 "multicomp:0603" H 1630 4600 20  0001 C CNN
-F 3 "" H 1569 4489 60  0001 C CNN
-F 4 "9330380" H 1969 4889 60  0001 C CNN "1st Source Part Number"
-F 5 "Farnell" H 1869 4789 60  0001 C CNN "1st Source"
-F 6 "MC0063W060311K" H 1769 4689 60  0001 C CNN "Manufacturer Part Number"
-F 7 "MULTICOMP" H 1669 4589 60  0001 C CNN "Manufacturer"
-	1    1600 4450
+P 3100 4450
+F 0 "R202" V 3108 4508 45  0000 L CNN
+F 1 "1K" V 3192 4508 45  0000 L CNN
+F 2 "multicomp:0603" H 3130 4600 20  0001 C CNN
+F 3 "" H 3069 4489 60  0001 C CNN
+F 4 "9330380" H 3469 4889 60  0001 C CNN "1st Source Part Number"
+F 5 "Farnell" H 3369 4789 60  0001 C CNN "1st Source"
+F 6 "MC0063W060311K" H 3269 4689 60  0001 C CNN "Manufacturer Part Number"
+F 7 "MULTICOMP" H 3169 4589 60  0001 C CNN "Manufacturer"
+	1    3100 4450
 	0    1    1    0
 $EndComp
 $Comp
-L GND #PWR201
+L GND #PWR203
 U 1 1 59B128CC
-P 1600 4750
-F 0 "#PWR201" H 1600 4500 50  0001 C CNN
-F 1 "GND" H 1605 4577 50  0000 C CNN
-F 2 "" H 1600 4750 50  0000 C CNN
-F 3 "" H 1600 4750 50  0000 C CNN
-	1    1600 4750
-	1    0    0    -1
-$EndComp
-Wire Wire Line
-	1600 4750 1600 4650
-Wire Wire Line
-	1600 4250 1600 4350
-Wire Wire Line
-	1600 3950 1600 3850
+P 3100 4700
+F 0 "#PWR203" H 3100 4450 50  0001 C CNN
+F 1 "GND" H 3105 4527 50  0000 C CNN
+F 2 "" H 3100 4700 50  0000 C CNN
+F 3 "" H 3100 4700 50  0000 C CNN
+	1    3100 4700
+	1    0    0    -1
+$EndComp
+Wire Wire Line
+	3100 4700 3100 4650
+Wire Wire Line
+	3100 4250 3100 4350
+Wire Wire Line
+	3100 3950 3100 3850
 Connection ~ 1600 3850
 Wire Wire Line
-	1600 4300 1700 4300
-Connection ~ 1600 4300
-Text HLabel 1700 4300 2    60   Output ~ 0
+	3100 4300 2600 4300
+Connection ~ 3100 4300
+Text HLabel 2600 4300 0    60   Output ~ 0
 VDD_SENSE
 $Comp
@@
 $EndComp
 Wire Wire Line
-	2900 3200 2450 3200
+	2750 3200 2450 3200
 Wire Wire Line
 	1500 2650 1500 3850
@@
 Connection ~ 1500 2750
 Wire Wire Line
-	2450 2700 2750 2700
+	2450 2700 3150 2700
 Wire Wire Line
 	2750 2700 2750 3200
-Connection ~ 2750 3200
+Connection ~ 3100 3850
+$Comp
+L CAP_EEE-FK1H470P C202
+U 1 1 5A13B69C
+P 3800 4050
+F 0 "C202" V 3708 4153 45  0000 L CNN
+F 1 "CAP_EEE-FK1H470P" V 3792 4153 45  0000 L CNN
+F 2 "usevolt:CAP_EEE-FK1H470P" H 3830 4200 20  0001 C CNN
+F 3 "http://industrial.panasonic.com/www-cgi/jvcr13pz.cgi?E+PZ+3+ABA0120+EEEFK1H470P+7+WW" H 3800 3990 60  0001 C CNN
+F 4 "667-EEE-FK1H470P" H 4400 4590 60  0001 C CNN "2nd Source Part Number"
+F 5 "Digi-Key" H 4100 4290 60  0001 C CNN "1st Source"
+F 6 "EEE-FK1H470P" H 4000 4190 60  0001 C CNN "Manufacturer Part Number"
+F 7 "Mouser" H 4300 4490 60  0001 C CNN "2nd Source"
+F 8 "Panasonic Electronic Components" H 3900 4090 60  0001 C CNN "Manufacturer"
+F 9 "PCE3815CT-ND" H 4200 4390 60  0001 C CNN "1st Source Part Number"
+	1    3800 4050
+	0    1    1    0
+$EndComp
+Connection ~ 3800 3850
+Connection ~ 2750 2700
+$Comp
+L DIODE_TVS_TPSMD28A D206
+U 1 1 5A13BC8E
+P 2900 2950
+F 0 "D206" V 2992 2882 45  0000 R CNN
+F 1 "DIODE_TVS_TPSMD28A" V 2908 2882 45  0000 R CNN
+F 2 "usevolt:DO-214AB" H 2930 3100 20  0001 C CNN
+F 3 "http://www.littelfuse.com/~/media/electronics/datasheets/tvs_diodes/littelfuse_tvs_diode_tpsmd_datasheet.pdf.pdf" H 3010 2960 60  0001 C CNN
+F 4 "Digi-Key" H 3310 3260 60  0001 C CNN "1st Source"
+F 5 "Littlefuse" H 3110 3060 60  0001 C CNN "Manufacturer"
+F 6 "TPSMD28A" H 3210 3160 60  0001 C CNN "Manufacturer Part Number"
+F 7 "F6570CT-ND" H 3410 3360 60  0001 C CNN "1st Source Part Number"
+	1    2900 2950
+	0    -1   -1   0
+$EndComp
+Wire Wire Line
+	2900 2750 2900 2700
+Connection ~ 2900 2700
+$Comp
+L GND #PWR202
+U 1 1 5A13BD77
+P 2900 3150
+F 0 "#PWR202" H 2900 2900 50  0001 C CNN
+F 1 "GND" H 2905 2977 50  0000 C CNN
+F 2 "" H 2900 3150 50  0000 C CNN
+F 3 "" H 2900 3150 50  0000 C CNN
+	1    2900 3150
+	1    0    0    -1
+$EndComp
+Wire Wire Line
+	2900 3150 2900 3050
 $EndSCHEMATC

Commit message: working revision in FM_6.6.1
Connections:
- wire segments 41 -> 40
Changed lines of the file:
@@
 LIBS:wurth_elektronik_LED
 LIBS:power
-LIBS:elt21300_kicad
 LIBS:yageo
 LIBS:esb-cache
@@
 	0    1    1    0
 $EndComp
-Wire Wire Line
-	8000 4950 8000 4250
-Wire Wire Line
-	6850 4950 6850 4150
-Connection ~ 8000 4950
-Wire Wire Line
-	6200 4950 6200 4150
-Connection ~ 6850 4950
-Wire Wire Line
-	5550 4950 5550 4050
-Connection ~ 6200 4950
-Wire Wire Line
-	3800 4950 3800 4150
-Connection ~ 5550 4950
-Wire Wire Line
-	3400 4950 3400 4150
-Connection ~ 3800 4950
-Wire Wire Line
-	2800 4150 2800 5150
-Connection ~ 3400 4950
-Connection ~ 2800 3850
-Connection ~ 3400 3850
-Wire Wire Line
-	8600 4950 8600 4150
-Wire Wire Line
-	8600 3600 8600 3850
-Wire Wire Line
-	8600 3850 8400 3850
-Wire Wire Line
-	6700 3850 7600 3850
-Connection ~ 6850 3850
-Wire Wire Line
-	5550 3850 6300 3850
-Connection ~ 6200 3850
-Wire Wire Line
-	6000 3950 6000 3850
-Connection ~ 6000 3850
-Wire Wire Line
-	5700 3950 5550 3950
-Wire Wire Line
-	5550 3750 6850 3750
-Wire Wire Line
-	6850 3600 6850 3850
-$Comp
-L +5V #PWR206
+$Comp
+L +5V #PWR07
 U 1 1 57B831F8
 P 6850 3600
-F 0 "#PWR206" H 6850 3450 50  0001 C CNN
+F 0 "#PWR07" H 6850 3450 50  0001 C CNN
 F 1 "+5V" H 6865 3773 50  0000 C CNN
 F 2 "" H 6850 3600 50  0000 C CNN
@@
 	1    0    0    -1
 $EndComp
-Connection ~ 6850 3750
-$Comp
-L +3V3 #PWR207
+$Comp
+L +3V3 #PWR08
 U 1 1 57B83259
 P 8600 3600
-F 0 "#PWR207" H 8600 3450 50  0001 C CNN
+F 0 "#PWR08" H 8600 3450 50  0001 C CNN
 F 1 "+3V3" H 8615 3773 50  0000 C CNN
 F 2 "" H 8600 3600 50  0000 C CNN
@@
 	1    0    0    -1
 $EndComp
-Wire Wire Line
-	1350 3850 1700 3850
-Wire Wire Line
-	3800 3700 4550 3700
-Wire Wire Line
-	4550 3700 4550 3750
 Text HLabel 7050 3600 2    60   Output ~ 0
 +5V
-Wire Wire Line
-	7050 3600 6850 3600
 Text HLabel 8750 3600 2    60   Output ~ 0
 +3V3
-Wire Wire Line
-	8750 3600 8600 3600
 Text HLabel 3150 2700 2    60   Output ~ 0
 VDD
 Text HLabel 2700 4950 0    60   Input ~ 0
 GND
-Connection ~ 2800 4950
 NoConn ~ 4550 3850
 NoConn ~ 4550 3950
 NoConn ~ 4550 4050
 $Comp
-L VDD #PWR204
+L VDD #PWR09
 U 1 1 57B9C56A
 P 3800 2100
-F 0 "#PWR204" H 3800 1950 50  0001 C CNN
+F 0 "#PWR09" H 3800 1950 50  0001 C CNN
 F 1 "VDD" H 3817 2273 50  0000 C CNN
 F 2 "" H 3800 2100 50  0000 C CNN
@@
 $EndComp
 $Comp
-L PWR_FLAG #FLG201
+L PWR_FLAG #FLG010
 U 1 1 57B9C59C
 P 3800 2300
-F 0 "#FLG201" H 3800 2395 50  0001 C CNN
+F 0 "#FLG010" H 3800 2395 50  0001 C CNN
 F 1 "PWR_FLAG" H 3800 2523 50  0000 C CNN
 F 2 "" H 3800 2300 50  0000 C CNN
@@
 	-1   0    0    1
 $EndComp
-Wire Wire Line
-	3800 2300 3800 2100
-$Comp
-L GND #PWR205
+$Comp
+L GND #PWR011
 U 1 1 57B9D351
 P 4300 2350
-F 0 "#PWR205" H 4300 2100 50  0001 C CNN
+F 0 "#PWR011" H 4300 2100 50  0001 C CNN
 F 1 "GND" H 4305 2177 50  0000 C CNN
 F 2 "" H 4300 2350 50  0000 C CNN
@@
 $EndComp
 $Comp
-L PWR_FLAG #FLG202
+L PWR_FLAG #FLG012
 U 1 1 57B9D3A1
 P 4300 2150
-F 0 "#FLG202" H 4300 2245 50  0001 C CNN
+F 0 "#FLG012" H 4300 2245 50  0001 C CNN
 F 1 "PWR_FLAG" H 4300 2374 50  0000 C CNN
 F 2 "" H 4300 2150 50  0000 C CNN
@@
 	1    0    0    -1
 $EndComp
-Wire Wire Line
-	4300 2150 4300 2350
-$Comp
-L GND #PWR201
+$Comp
+L GND #PWR013
 U 1 1 57CF1F5E
 P 2800 5150
-F 0 "#PWR201" H 2800 4900 50  0001 C CNN
+F 0 "#PWR013" H 2800 4900 50  0001 C CNN
 F 1 "GND" H 2805 4977 50  0000 C CNN
 F 2 "" H 2800 5150 50  0000 C CNN
@@
 	1    0    0    -1
 $EndComp
-Wire Wire Line
-	3800 3850 3800 3700
-Connection ~ 1500 3850
-Wire Wire Line
-	2700 3850 3800 3850
 $Comp
 L IND_744045210 L201
@@
 	1    0    0    -1
 $EndComp
-Wire Wire Line
-	2000 3850 2300 3850
-Wire Wire Line
-	2700 4950 8600 4950
 $Comp
 L DIODE_RS07J-GS18 D201
@@
 L 10K R201
 U 1 1 59B1277F
-P 3100 4050
-F 0 "R201" V 3108 4108 45  0000 L CNN
-F 1 "10K" V 3192 4108 45  0000 L CNN
-F 2 "multicomp:0603" H 3130 4200 20  0001 C CNN
-F 3 "http://www.farnell.com/datasheets/1788326.pdf?_ga=1.214208087.1948984246.1460023966" H 3069 4089 60  0001 C CNN
-F 4 "9330399" H 3469 4489 60  0001 C CNN "1st Source Part Number"
-F 5 "Farnell" H 3369 4389 60  0001 C CNN "1st Source"
-F 6 "MC0063W0603110K" H 3269 4289 60  0001 C CNN "Manufacturer Part Number"
-F 7 "MULTICOMP" H 3169 4189 60  0001 C CNN "Manufacturer"
-	1    3100 4050
+P 1500 4350
+F 0 "R201" V 1508 4408 45  0000 L CNN
+F 1 "10K" V 1592 4408 45  0000 L CNN
+F 2 "multicomp:0603" H 1530 4500 20  0001 C CNN
+F 3 "http://www.farnell.com/datasheets/1788326.pdf?_ga=1.214208087.1948984246.1460023966" H 1469 4389 60  0001 C CNN
+F 4 "9330399" H 1869 4789 60  0001 C CNN "1st Source Part Number"
+F 5 "Farnell" H 1769 4689 60  0001 C CNN "1st Source"
+F 6 "MC0063W0603110K" H 1669 4589 60  0001 C CNN "Manufacturer Part Number"
+F 7 "MULTICOMP" H 1569 4489 60  0001 C CNN "Manufacturer"
+	1    1500 4350
 	0    1    1    0
 $EndComp
@@
 L 1K R202
 U 1 1 59B12803
-P 3100 4450
-F 0 "R202" V 3108 4508 45  0000 L CNN
-F 1 "1K" V 3192 4508 45  0000 L CNN
-F 2 "multicomp:0603" H 3130 4600 20  0001 C CNN
-F 3 "" H 3069 4489 60  0001 C CNN
-F 4 "9330380" H 3469 4889 60  0001 C CNN "1st Source Part Number"
-F 5 "Farnell" H 3369 4789 60  0001 C CNN "1st Source"
-F 6 "MC0063W060311K" H 3269 4689 60  0001 C CNN "Manufacturer Part Number"
-F 7 "MULTICOMP" H 3169 4589 60  0001 C CNN "Manufacturer"
-	1    3100 4450
+P 1500 4750
+F 0 "R202" V 1508 4808 45  0000 L CNN
+F 1 "1K" V 1592 4808 45  0000 L CNN
+F 2 "multicomp:0603" H 1530 4900 20  0001 C CNN
+F 3 "" H 1469 4789 60  0001 C CNN
+F 4 "9330380" H 1869 5189 60  0001 C CNN "1st Source Part Number"
+F 5 "Farnell" H 1769 5089 60  0001 C CNN "1st Source"
+F 6 "MC0063W060311K" H 1669 4989 60  0001 C CNN "Manufacturer Part Number"
+F 7 "MULTICOMP" H 1569 4889 60  0001 C CNN "Manufacturer"
+	1    1500 4750
 	0    1    1    0
 $EndComp
 $Comp
-L GND #PWR203
+L GND #PWR014
 U 1 1 59B128CC
-P 3100 4700
-F 0 "#PWR203" H 3100 4450 50  0001 C CNN
-F 1 "GND" H 3105 4527 50  0000 C CNN
-F 2 "" H 3100 4700 50  0000 C CNN
-F 3 "" H 3100 4700 50  0000 C CNN
-	1    3100 4700
-	1    0    0    -1
-$EndComp
-Wire Wire Line
-	3100 4700 3100 4650
-Wire Wire Line
-	3100 4250 3100 4350
-Wire Wire Line
-	3100 3950 3100 3850
-Connection ~ 1600 3850
-Wire Wire Line
-	3100 4300 2600 4300
-Connection ~ 3100 4300
-Text HLabel 2600 4300 0    60   Output ~ 0
+P 1500 5000
+F 0 "#PWR014" H 1500 4750 50  0001 C CNN
+F 1 "GND" H 1505 4827 50  0000 C CNN
+F 2 "" H 1500 5000 50  0000 C CNN
+F 3 "" H 1500 5000 50  0000 C CNN
+	1    1500 5000
+	1    0    0    -1
+$EndComp
+Text HLabel 1450 4600 0    60   Output ~ 0
 VDD_SENSE
 $Comp
@@
 	1    0    0    -1
 $EndComp
-Wire Wire Line
-	2750 3200 2450 3200
-Wire Wire Line
-	1500 2650 1500 3850
-Wire Wire Line
-	1500 3150 1650 3150
-Wire Wire Line
-	1650 3250 1500 3250
-Connection ~ 1500 3250
 $Comp
 L SCHOTTKY_DIODE_V40PW10C D205
@@
 	1    0    0    -1
 $EndComp
-Wire Wire Line
-	1500 2750 1650 2750
-Connection ~ 1500 3150
-Wire Wire Line
-	1500 2650 1650 2650
-Connection ~ 1500 2750
-Wire Wire Line
-	2450 2700 3150 2700
-Wire Wire Line
-	2750 2700 2750 3200
-Connection ~ 3100 3850
 $Comp
 L CAP_EEE-FK1H470P C202
@@
 	0    1    1    0
 $EndComp
-Connection ~ 3800 3850
-Connection ~ 2750 2700
 $Comp
 L DIODE_TVS_TPSMD28A D206
@@
 	0    -1   -1   0
 $EndComp
-Wire Wire Line
-	2900 2750 2900 2700
-Connection ~ 2900 2700
-$Comp
-L GND #PWR202
+$Comp
+L GND #PWR015
 U 1 1 5A13BD77
 P 2900 3150
-F 0 "#PWR202" H 2900 2900 50  0001 C CNN
+F 0 "#PWR015" H 2900 2900 50  0001 C CNN
 F 1 "GND" H 2905 2977 50  0000 C CNN
 F 2 "" H 2900 3150 50  0000 C CNN
@@
 $EndComp
 Wire Wire Line
+	8000 4950 8000 4250
+Wire Wire Line
+	6850 4950 6850 4150
+Connection ~ 8000 4950
+Wire Wire Line
+	6200 4950 6200 4150
+Connection ~ 6850 4950
+Wire Wire Line
+	5550 4950 5550 4050
+Connection ~ 6200 4950
+Wire Wire Line
+	3800 4950 3800 4150
+Connection ~ 5550 4950
+Wire Wire Line
+	3400 4950 3400 4150
+Connection ~ 3800 4950
+Wire Wire Line
+	2800 4150 2800 5150
+Connection ~ 3400 4950
+Connection ~ 2800 3850
+Connection ~ 3400 3850
+Wire Wire Line
+	8600 4950 8600 4150
+Wire Wire Line
+	8600 3600 8600 3850
+Wire Wire Line
+	8600 3850 8400 3850
+Wire Wire Line
+	6700 3850 7600 3850
+Connection ~ 6850 3850
+Wire Wire Line
+	5550 3850 6300 3850
+Connection ~ 6200 3850
+Wire Wire Line
+	6000 3950 6000 3850
+Connection ~ 6000 3850
+Wire Wire Line
+	5700 3950 5550 3950
+Wire Wire Line
+	5550 3750 6850 3750
+Wire Wire Line
+	6850 3600 6850 3850
+Connection ~ 6850 3750
+Wire Wire Line
+	1350 3850 1700 3850
+Wire Wire Line
+	3800 3700 4550 3700
+Wire Wire Line
+	4550 3700 4550 3750
+Wire Wire Line
+	7050 3600 6850 3600
+Wire Wire Line
+	8750 3600 8600 3600
+Connection ~ 2800 4950
+Wire Wire Line
+	3800 2300 3800 2100
+Wire Wire Line
+	4300 2150 4300 2350
+Wire Wire Line
+	3800 3850 3800 3700
+Connection ~ 1500 3850
+Wire Wire Line
+	2700 3850 3800 3850
+Wire Wire Line
+	2000 3850 2300 3850
+Wire Wire Line
+	2700 4950 8600 4950
+Wire Wire Line
+	1500 5000 1500 4950
+Wire Wire Line
+	1500 4550 1500 4650
+Wire Wire Line
+	1500 4600 1450 4600
+Connection ~ 1500 4600
+Wire Wire Line
+	2750 3200 2450 3200
+Wire Wire Line
+	1500 2650 1500 4250
+Wire Wire Line
+	1500 3150 1650 3150
+Wire Wire Line
+	1650 3250 1500 3250
+Connection ~ 1500 3250
+Wire Wire Line
+	1500 2750 1650 2750
+Connection ~ 1500 3150
+Wire Wire Line
+	1500 2650 1650 2650
+Connection ~ 1500 2750
+Wire Wire Line
+	2450 2700 3150 2700
+Wire Wire Line
+	2750 2700 2750 3200
+Connection ~ 3800 3850
+Connection ~ 2750 2700
+Wire Wire Line
+	2900 2750 2900 2700
+Connection ~ 2900 2700
+Wire Wire Line
 	2900 3150 2900 3050
