File: hw/bts6133d.sch (KiCad schematic (older format))
At the start: 3 parts, among them U601 BTS6133D

Commit message: flyback diodes added for solenoid outputs
Changed lines of the file:
@@
 AR Path="/5A13680F/59D7DBA1" Ref="U1502"  Part="1"
 AR Path="/5A14370A/59D7DBA1" Ref="U1602"  Part="1"
-F 0 "U901" H 5050 3547 60  0000 C CNN
+F 0 "U1201" H 5050 3547 60  0000 C CNN
 F 1 "BTS6133D" H 5050 3441 60  0000 C CNN
 F 2 "usevolt:DPAK-5" H 4800 3700 60  0001 C CNN
@@
 AR Path="/5A13680F/59D7D931" Ref="R1503"  Part="1"
 AR Path="/5A14370A/59D7D931" Ref="R1603"  Part="1"
-F 0 "R902" H 4200 3484 45  0000 C CNN
+F 0 "R1202" H 4200 3484 45  0000 C CNN
 F 1 "560" H 4200 3400 45  0000 C CNN
 F 2 "yageo:0603" H 4180 3450 20  0001 C CNN
@@
 AR Path="/5A01A445/59D7E637" Ref="#PWR702"  Part="1"
 AR Path="/5A01AB59/59D7E637" Ref="#PWR802"  Part="1"
-AR Path="/5A120DD2/59D7E637" Ref="#PWR902"  Part="1"
-AR Path="/5A12FF64/59D7E637" Ref="#PWR1102"  Part="1"
-AR Path="/5A130D3E/59D7E637" Ref="#PWR1202"  Part="1"
-AR Path="/5A1349CF/59D7E637" Ref="#PWR1302"  Part="1"
-AR Path="/5A1358B0/59D7E637" Ref="#PWR1402"  Part="1"
-AR Path="/5A13680F/59D7E637" Ref="#PWR1502"  Part="1"
-AR Path="/5A14370A/59D7E637" Ref="#PWR1602"  Part="1"
+AR Path="/5A120DD2/59D7E637" Ref="#PWR602"  Part="1"
+AR Path="/5A12FF64/59D7E637" Ref="#PWR802"  Part="1"
+AR Path="/5A130D3E/59D7E637" Ref="#PWR902"  Part="1"
+AR Path="/5A1349CF/59D7E637" Ref="#PWR1002"  Part="1"
+AR Path="/5A1358B0/59D7E637" Ref="#PWR1102"  Part="1"
+AR Path="/5A13680F/59D7E637" Ref="#PWR1202"  Part="1"
+AR Path="/5A14370A/59D7E637" Ref="#PWR1302"  Part="1"
 F 0 "#PWR902" H 4600 2850 50  0001 C CNN
 F 1 "VDD" H 4617 3173 50  0000 C CNN
@@
 AR Path="/5A01A445/5A014ACD" Ref="#PWR701"  Part="1"
 AR Path="/5A01AB59/5A014ACD" Ref="#PWR801"  Part="1"
-AR Path="/5A120DD2/5A014ACD" Ref="#PWR901"  Part="1"
-AR Path="/5A12FF64/5A014ACD" Ref="#PWR1101"  Part="1"
-AR Path="/5A130D3E/5A014ACD" Ref="#PWR1201"  Part="1"
-AR Path="/5A1349CF/5A014ACD" Ref="#PWR1301"  Part="1"
-AR Path="/5A1358B0/5A014ACD" Ref="#PWR1401"  Part="1"
-AR Path="/5A13680F/5A014ACD" Ref="#PWR1501"  Part="1"
-AR Path="/5A14370A/5A014ACD" Ref="#PWR1601"  Part="1"
+AR Path="/5A120DD2/5A014ACD" Ref="#PWR601"  Part="1"
+AR Path="/5A12FF64/5A014ACD" Ref="#PWR801"  Part="1"
+AR Path="/5A130D3E/5A014ACD" Ref="#PWR901"  Part="1"
+AR Path="/5A1349CF/5A014ACD" Ref="#PWR1001"  Part="1"
+AR Path="/5A1358B0/5A014ACD" Ref="#PWR1101"  Part="1"
+AR Path="/5A13680F/5A014ACD" Ref="#PWR1201"  Part="1"
+AR Path="/5A14370A/5A014ACD" Ref="#PWR1301"  Part="1"
 F 0 "#PWR901" H 3850 3350 50  0001 C CNN
 F 1 "GND" H 3855 3427 50  0000 C CNN
@@
 AR Path="/5A13680F/5A058D94" Ref="R1502"  Part="1"
 AR Path="/5A14370A/5A058D94" Ref="R1602"  Part="1"
-F 0 "R901" V 3608 3408 45  0000 L CNN
+F 0 "R1201" V 3608 3408 45  0000 L CNN
 F 1 "1K" V 3692 3408 45  0000 L CNN
 F 2 "yageo:0603" H 3630 3500 20  0001 C CNN
