File: hw/PT100.sch (KiCad schematic (older format))
At the start: 10 parts, among them U701 OPAMP_MCP6002

Commit message: 4.2.0 created, with working propo solenoid pump driver
Parts:
- removed C701: 100nF, kemet:0603, symbol 100nF
- removed R701, R702: 1K, yageo:0603, symbol 1K
- removed R703, R704, R705, R706: 10K, yageo:0603, symbol 10K
- removed R707, R708: 1K5, yageo:0603, symbol 1K5
- removed U701: OPAMP_MCP6002, usevolt:SOIC8, symbol OPAMP_MCP6002
- added R1401: 10K, multicomp:0603, symbol 10K
- added U1401: ZXCT1086, usevolt:SOT-25, symbol ZXCT1086
Connections:
- net labels added: SENSOR, VOUT
- net labels removed: SENSOR1, SENSOR2, VOUT1, VOUT2
- wire segments 27 -> 10

Commit message: hw bugs fixed from 4.2.0 revsion
Parts:
- removed R1401: 10K, multicomp:0603, symbol 10K
- removed U1401: ZXCT1086, usevolt:SOT-25, symbol ZXCT1086
- added C701: 100nF, kemet:0603, symbol 100nF
- added R701, R702: 1K, yageo:0603, symbol 1K
- added R703, R704, R705, R706: 10K, yageo:0603, symbol 10K
- added R707, R708: 1K5, yageo:0603, symbol 1K5
- added U701: OPAMP_MCP6002, usevolt:SOIC8, symbol OPAMP_MCP6002
Connections:
- net labels added: SENSOR1, SENSOR2, VOUT1, VOUT2
- net labels removed: SENSOR, VOUT
- wire segments 10 -> 27

Commit message: starting to redraw the pcb as a smaller (icu enclosure)
Parts:
- C701: symbol 100nF -> kemet:100nF
- R701, R702: symbol 1K -> yageo:1K
- R703, R704, R705, R706: symbol 10K -> yageo:10K
- R707, R708: symbol 1K5 -> yageo:1K5
- U701: symbol OPAMP_MCP6002 -> usevolt:OPAMP_MCP6002
Changed lines of the file:
@@
-EESchema Schematic File Version 2
-LIBS:esb-rescue
-LIBS:kemet
-LIBS:usevolt
-LIBS:wurth_elektronik_LED
-LIBS:power
-LIBS:yageo
+EESchema Schematic File Version 4
 LIBS:esb-cache
 EELAYER 26 0
@@
 VOUT2
 $Comp
-L +3V3 #PWR026
+L power:+3V3 #PWR026
 U 1 1 59EDDEDF
 P 4050 3350
@@
 $EndComp
 $Comp
-L GND #PWR027
+L power:GND #PWR027
 U 1 1 59EDDEF8
 P 4050 4000
@@
 	4050 3850 4300 3850
 $Comp
-L 100nF C701
+L kemet:100nF C701
 U 1 1 59EDDF13
 P 4050 3700
@@
 $EndComp
 $Comp
-L OPAMP_MCP6002 U701
+L usevolt:OPAMP_MCP6002 U701
 U 1 1 59EDF729
 P 4550 3550
@@
 	5050 3750 5850 3750
 $Comp
-L +3V3 #PWR028
+L power:+3V3 #PWR028
 U 1 1 59EDF8B8
 P 7000 3000
@@
 	5050 3850 6650 3850
 $Comp
-L 10K R705
+L yageo:10K R705
 U 1 1 59EDFACF
 P 6750 3450
@@
 $EndComp
 $Comp
-L 10K R706
+L yageo:10K R706
 U 1 1 59EDFB0E
 P 6750 3850
@@
 $EndComp
 $Comp
-L 10K R703
+L yageo:10K R703
 U 1 1 59EE04D0
 P 5500 3550
@@
 	5050 3550 5400 3550
 $Comp
-L 1K R701
+L yageo:1K R701
 U 1 1 59EE059A
 P 5300 3650
@@
 	5150 3650 5150 3550
 $Comp
-L 10K R704
+L yageo:10K R704
 U 1 1 59EE0699
 P 5500 3950
@@
 $EndComp
 $Comp
-L 1K R702
+L yageo:1K R702
 U 1 1 59EE06D8
 P 5300 4050
@@
 Connection ~ 5150 3950
 $Comp
-L GND #PWR029
+L power:GND #PWR029
 U 1 1 59EE07A1
 P 6250 4100
@@
 	6950 3850 7450 3850
 $Comp
-L 1K5 R708
+L yageo:1K5 R708
 U 1 1 59EE17CE
 P 7100 3700
@@
 $EndComp
 $Comp
-L 1K5 R707
+L yageo:1K5 R707
 U 1 1 59EE1849
 P 7100 3300
